File: Hardware/Pyrologger_V3_KiCad/Pyrologger_V3.sch (KiCad schematic (older format))
At the start: 9 parts, among them J1 RJ12, P1 CONN_02X14, P2 CONN_02X14, U1 MICRO-SDCARD_MICRO-SDCARD, U2 TEENSY_3.1_BASIC_TEENSY_3.1_B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

Commit message: finished off the kicad board file and starting to work on the arduino code
Parts:
- R1, R2, R3: footprint Resistors_SMD:R_1206_HandSoldering -> Resistors_SMD:R_0805_HandSoldering
Changed lines of the file:
@@
 F 0 "R3" V 4480 1400 40  0000 C CNN
 F 1 "4.7K" V 4407 1401 40  0000 C CNN
-F 2 "Resistors_SMD:R_1206_HandSoldering" V 4330 1400 30  0001 C CNN
+F 2 "Resistors_SMD:R_0805_HandSoldering" V 4330 1400 30  0001 C CNN
 F 3 "" H 4400 1400 30  0000 C CNN
 	1    4400 1400
@@
 F 0 "R1" V 2330 1100 40  0000 C CNN
 F 1 "10K" V 2257 1101 40  0000 C CNN
-F 2 "Resistors_SMD:R_1206_HandSoldering" V 2180 1100 30  0001 C CNN
+F 2 "Resistors_SMD:R_0805_HandSoldering" V 2180 1100 30  0001 C CNN
 F 3 "" H 2250 1100 30  0000 C CNN
 	1    2250 1100
@@
 F 0 "R2" V 2880 2850 40  0000 C CNN
 F 1 "330 " V 2807 2851 40  0000 C CNN
-F 2 "Resistors_SMD:R_1206_HandSoldering" V 2730 2850 30  0001 C CNN
+F 2 "Resistors_SMD:R_0805_HandSoldering" V 2730 2850 30  0001 C CNN
 F 3 "" H 2800 2850 30  0000 C CNN
 	1    2800 2850
